Commit message: 

File: models/Sirius3/Sirius3.urdf (robot description, URDF)
Before this commit: robot Sirius3, 4 links, 3 joints
Links:
- removed link Left-Wheel-v1
- removed link Right-Wheel-v1
- removed link Sirius3-body-v2
- added link base_footprint
- added link left_wheel, mass 26.684250609189966; collision mesh filename=file:///home/kotantu-desktop/ros2_ws/src/urdf_viewer/models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 scale=0.001 0.001 0.001; visual mesh filename=file:///home/kotantu-desktop/ros2_ws/src/urdf_viewer/models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 scale=0.001 0.001 0.001
- added link right_wheel, mass 26.680591288269447; collision mesh filename=file:///home/kotantu-desktop/ros2_ws/src/urdf_viewer/models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 scale=0.001 0.001 0.001; visual mesh filename=file:///home/kotantu-desktop/ros2_ws/src/urdf_viewer/models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 scale=0.001 0.001 0.001
- link base_link: mass None -> 55.92590679361776; geometry collision mesh filename=file:///home/kotantu-desktop/ros2_ws/src/urdf_viewer/models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 scale=0.001 0.001 0.001; visual mesh filename=file:///home/kotantu-desktop/ros2_ws/src/urdf_viewer/models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 scale=0.001 0.001 0.001
Joints:
- removed joint base_link_to_body
- removed joint rev1
- removed joint rev2
- added joint footprint_to_base: type fixed, parent base_footprint, child base_link, origin xyz=0 0 0 rpy=0 0 0
- added joint left_wheel_joint: type continuous, parent base_link, child left_wheel, origin xyz=0.18100000000000002 -0.0014818300000000002 0.13236434 rpy=-3.141592653589793 -1.5707963267948966 0, axis 0.0 0.0 1.0
- added joint right_wheel_joint: type continuous, parent base_link, child right_wheel, origin xyz=-0.18100000000000002 -0.0014818300000000002 0.1325 rpy=-0.0 -1.5707963267948966 0, axis 0.0 0.0 1.0

Commit message: fix joint state publisher bug

File: models/Sirius3/Sirius3.urdf (robot description, URDF)
Before this commit: robot Sirius3, 4 links, 3 joints
Joints:
- joint left_wheel_joint: limit (none) -> effort=100 velocity=100
- joint right_wheel_joint: limit (none) -> effort=100 velocity=100

Commit message: teleop

File: models/Sirius3/Sirius3.urdf (robot description, URDF)
Before this commit: robot Sirius3, 4 links, 3 joints
Joints:
- joint right_wheel_joint: axis 0.0 0.0 1.0 -> 0.0 0.0 -1.0
